File: hardware/0.1/usb.sch (KiCad schematic (older format))
At the start: 43 parts, among them J3 USB_A, J4 USB_A, J5 USB_A, U3 TS3USB30, U4 TPS211x, U5 CY7C65632-28LTXCT, Y1 12MHz

Commit message: add mcu + 2x4 switches + icsp
Parts:
- renumbered C16 to C10, C13 to C11, C9 to C12, C10 to C13, C5 to C14, C6 to C15, C7 to C16, C8 to C17, C11 to C18, C12 to C19, C15 to C20, C1 to C21, C3 to C22, C2 to C7, C4 to C8, C14 to C9, D2 to D10, D1 to D9, FB5 to FB3, FB6 to FB5, FB3 to FB6, J3 to J5, J5 to J6, R1 to R10, R4 to R11, R6 to R12, R10 to R13, R11 to R14, R12 to R15, R9 to R16, R8 to R4, R13 to R5, R2 to R6, R3 to R7, R5 to R8, R7 to R9, U3 to U5, U5 to U6, Y1 to Y2

Commit message: Update jkl & footprints
USBA / Kailh Choc / ATMEGA32U4-AU
Parts:
- J4, J5, J6: footprint josh-connectors:USB_A_Molex_67643_Horizontal -> josh-connectors:USB_A_U234-051N-3GRA035-5
Changed lines of the file:
@@
 F 0 "J6" H 10950 6200 50  0000 R CNN
 F 1 "USB_A" H 10950 6100 50  0000 R CNN
-F 2 "josh-connectors:USB_A_Molex_67643_Horizontal" H 10900 5700 50  0001 C CNN
+F 2 "josh-connectors:USB_A_U234-051N-3GRA035-5" H 10900 5700 50  0001 C CNN
 F 3 " ~" H 10900 5700 50  0001 C CNN
 	1    10750 5750
@@
 F 0 "J5" H 9650 6200 50  0000 R CNN
 F 1 "USB_A" H 9650 6100 50  0000 R CNN
-F 2 "josh-connectors:USB_A_Molex_67643_Horizontal" H 9600 5700 50  0001 C CNN
+F 2 "josh-connectors:USB_A_U234-051N-3GRA035-5" H 9600 5700 50  0001 C CNN
 F 3 " ~" H 9600 5700 50  0001 C CNN
 	1    9450 5750
@@
 F 0 "J4" H 10900 4900 50  0000 R CNN
 F 1 "USB_A" H 10900 4800 50  0000 R CNN
-F 2 "josh-connectors:USB_A_Molex_67643_Horizontal" H 10850 4400 50  0001 C CNN
+F 2 "josh-connectors:USB_A_U234-051N-3GRA035-5" H 10850 4400 50  0001 C CNN
 F 3 " ~" H 10850 4400 50  0001 C CNN
 	1    10700 4450

Commit message: Switch to VSON TS3USB221E for easier routing
Parts:
- U5: value TS3USB30 -> TS3USB221E; footprint josh-dfn-qfn:UQFN-10_1.4x1.8_Pitch0.4mm -> Package_SON:VSON-10-1EP_3x3mm_P0.5mm_EP1.65x2.4mm_ThermalVias; symbol josh-ic:TS3USB30 -> josh-ic:TS3USB221E
Connections:
- net +3.3VA: now also U5.10 (VCC); no longer U5.9 (VCC)
- net GND: now also U5.11 (EXP), U5.5 (GND); no longer U5.4 (GND)
- net UP_USB_N: now also U5.7 (D-); no longer U5.5 (D-)
- net UP_USB_P: now also U5.8 (D+); no longer U5.3 (D+)
- net USB_1_D-: now also U5.2 (D1-); no longer U5.7 (D1-)
- net USB_2_D+: now also U5.3 (D2+); no longer U5.2 (D2+)
- net USB_2_D-: now also U5.4 (D2-); no longer U5.6 (D2-)
- net at R10.1, R11.2: now also U5.9 (SEL); no longer U5.10 (SEL)
- net at R12.1: now also U5.6 (~OE); no longer U5.8 (~OE)
Changed lines of the file:
@@
 $EndComp
 $Comp
-L josh-ic:TS3USB30 U5
+L josh-ic:TS3USB221E U5
 U 1 1 5FBC75B1
 P 3900 3750
 F 0 "U5" H 3700 3850 50  0000 C CNN
-F 1 "TS3USB30" H 3850 3750 50  0000 C CNN
-F 2 "josh-dfn-qfn:UQFN-10_1.4x1.8_Pitch0.4mm" H 3900 3750 50  0001 C CNN
+F 1 "TS3USB221E" H 3850 3750 50  0000 C CNN
+F 2 "Package_SON:VSON-10-1EP_3x3mm_P0.5mm_EP1.65x2.4mm_ThermalVias" H 3900 3750 50  0001 C CNN
 F 3 "" H 3900 3750 50  0001 C CNN
 	1    3900 3750
@@
 	4450 1600 4450 1700
 Connection ~ 4450 1700
+Wire Wire Line
+	4250 4350 4300 4350
+Wire Wire Line
+	4300 4350 4300 4450
+Connection ~ 4300 4450
 $EndSCHEMATC
